File: esp-prog/SMD/esp-prog.kicad_pcb (KiCad board)
At the start: 2 copper layers, 30 x 19 mm, 9 parts, among them J1 Conn_01x07_Female, J2 Conn_02x03_Odd_Even, Q1 BC847, Q2 BC847

Commit message: add PDF output for ESP-Prog
Parts:
- removed QR*****: www.schwingen.org, MS_Mechanical:QR_schwingen_Silk
- Q1, Q2: value BC847 -> BCW33
- R1, R2: value 10k -> 8.2k
- R3, R4: value 100 -> 390
