File: YOGA_GPIB/yoga_v2.kicad_pcb (KiCad board)
At the start: 2 copper layers, 85 x 56 mm, 85 parts, among them J1 Conn_01x01_Female, J2 Conn_01x01_Female, J3 Conn_02x13_Odd_Even, J4 Conn_02x12_GPIB_PCB, J5 Raspberry_Pi_2_3, J6 Conn_01x10, J7 Conn_01x04, J8 22-23-2031, J9 Conn_01x05, Q1 BCW33, Q2 BCW30, Q3 BSS138, Q4 BSS138, U1 TPS62932, U2 LSF0108, U3 LSF0108, U4 24LC64, U5 ADM3202ARU, U6 SP385E

Commit message: YOGA_GPIB: update LED resistors and wiring documentation
Parts:
- R11: value 1K -> 4.7k
- R13: value 1K -> 680
- R2: value 4.7 -> 4.7
